File: hardware/NeuralCard.kicad_pcb (KiCad board)
At the start: 2 copper layers, 85.6 x 54 mm, 66 parts, among them J1 ProgPads, J2 TYPE-C-31-M-12, Q1 AO3401A, SW1 SW-SMD_4P-L5.1-W5.1-P3.70-LS6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, SW2 SW-SMD_4P-L5.1-W5.1-P3.70-LS6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, SW3 SW_SPDT_Shouhan_MSK12C02, U1 WIRELM-SMD_ESP32-S3-WROOM-1, U2 LGA-14_L3.0-W2.5-P0.50-TL, U3 ME6211C33M5G-N, U4 SO-8_L4.9-W3.9-P1.27-LS5.9-BL, U5 USBLC6-2SC6

Commit message: regenerate fab package
Other:
- board text added: "CR2032 ·"
- board text removed: "CR2032 · + side out"
- board text removed: "FLASH: hold BOOT · tap RST · release BOOT"
- board text removed: "NeuralCard v2.3.1 · princetekki.com"
- board text removed: "OSHW · github.com/Brillar0101"
