File: hardware/NeuralCard.kicad_sch (KiCad schematic)
At the start: 63 parts, among them J1 ProgPads, J2 TYPE-C-31-M-12, Q1 AO3401A, SW1 SW_PUSH, SW2 SW_PUSH, SW3 MSK12C02, U1 ESP32-S3-WROOM-1, U2 LSM6DS3TR-C, U3 ME6211C33M5G-N, U4 ST25DV04KC-IE6S3, U5 USBLC6-2SC6

Commit message: add part sourcing alternates
Parts:
- BT1: Sourcing (none) -> Shenzhen local stock -- PCBWay's preferred channel. Land pa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
- C1, C10, C11, C2, C3, C4, C5, C6, C7, C8, C9, R1, R10, R11, R12, R13, R14, R2, R3, R4, R5, R6, R9: Sourcing (none) -> PCBWay house stock acceptable -- any equivalent part, same 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
- C12: Sourcing (none) -> PCBWay house stock acceptable. MUST be C0G/NP0 dielectric -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
- D1, D10, D11, D12, D13, D14, D15, D16, D17, D18, D19, D2, D20, D21, D22, D23, D24, D3, D4, D5, D6, D7, D8, D9: Sourcing (none) -> Shenzhen local stock -- PCBWay's preferred channel. Any 060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
- J2: Alt MPN (none) -> U262-161N-4BVC11; Alt Mfr (none) -> XKB Connectivity; Sourcing (none) -> Shenzhen local stock -- PCBWay's preferred channel. Alterna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
- Q1: Alt MPN (none) -> DMG2301L; Alt Mfr (none) -> Diodes Incorporated; Sourcing (none) -> Global distributor (Digi-Key / Mouser / LCSC). Any -30V P-c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
- R7, R8: Sourcing (none) -> PCBWay house stock acceptable. 5.1k is FIXED by the USB-C s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
- SW1, SW2: Sourcing (none) -> Shenzhen local stock -- PCBWay's preferred channel. Any 4-p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
- SW3: Sourcing (none) -> Shenzhen local stock -- PCBWay's preferred channel. NO SUBS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
- U1: Alt MPN (none) -> ESP32-S3-WROOM-1-N16R8; Alt Mfr (none) -> Espressif Systems; Sourcing (none) -> Global distributor (Digi-Key / Mouser / LCSC). N16R8 is an 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
- U2: Sourcing (none) -> Global distributor (Digi-Key / Mouser / LCSC). NO SUBSTITUT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
- U3: Alt MPN (none) -> AP2112K-3.3TRG1; Alt Mfr (none) -> Diodes Incorporated; Sourcing (none) -> China-market part, NOT stocked at Digi-Key/Mouser. Shenzhen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
- U4: Alt MPN (none) -> ST25DV04K-IER6S3; Alt Mfr (none) -> STMicroelectronics; Sourcing (none) -> Global distributor (Digi-Key / Mouser / LCSC). Fitted part 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
- U5: Sourcing (none) -> Global distributor (Digi-Key / Mouser / LCSC). Deep stock e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

Commit message: rename part libraries
Parts:
- BT1: footprint JLC:BAT-TH_CR2032-BS-6-1 -> Parts:BAT-TH_CR2032-BS-6-1; symbol JLC:CR2032-BS-6-1 -> Parts:CR2032-BS-6-1
- D1, D10, D11, D12, D13, D14, D15, D16, D17, D18, D19, D2, D20, D21, D22, D23, D24, D3, D4, D5, D6, D7, D8, D9: footprint JLC:LED-SMD_L1.6-W0.8-R-RD -> Parts:LED-SMD_L1.6-W0.8-R-RD
- J2: footprint JLC:USB-C_SMD-TYPE-C-31-M-12_1 -> Parts:USB-C_SMD-TYPE-C-31-M-12_1; symbol JLC:TYPE-C-31-M-12 -> Parts:TYPE-C-31-M-12
- Q1: footprint JLC:SOT-23_L2.9-W1.3-P1.90-LS2.4-BR -> Parts:SOT-23_L2.9-W1.3-P1.90-LS2.4-BR; symbol JLC:AO3401A -> Parts:AO3401A
- SW1, SW2: footprint JLC:SW-SMD_4P-L5.1-W5.1-P3.70-LS6.5-TL_H1.5 -> Parts:SW-SMD_4P-L5.1-W5.1-P3.70-LS6.5-TL_H1.5; symbol JLC:TS-1187A-B-A-B -> Parts:TS-1187A-B-A-B
- U1: footprint JLC:WIRELM-SMD_ESP32-S3-WROOM-1 -> Parts:WIRELM-SMD_ESP32-S3-WROOM-1; symbol JLC:ESP32-S3-WROOM-1 -> Parts:ESP32-S3-WROOM-1
- U2: footprint JLC:LGA-14_L3.0-W2.5-P0.50-TL -> Parts:LGA-14_L3.0-W2.5-P0.50-TL; symbol JLC:LSM6DS3TR-C -> Parts:LSM6DS3TR-C
- U3: footprint JLC:SOT-23-5_L3.0-W1.7-P0.95-LS2.8-BL -> Parts:SOT-23-5_L3.0-W1.7-P0.95-LS2.8-BL; symbol JLC:ME6211C33M5G-N -> Parts:ME6211C33M5G-N
- U5: footprint JLC:SOT-23-6_L2.9-W1.6-P0.95-LS2.8-BL -> Parts:SOT-23-6_L2.9-W1.6-P0.95-LS2.8-BL; symbol JLC:USBLC6-2SC6 -> Parts:USBLC6-2SC6
Changed lines of the file:
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@@
 	)
 	(symbol
-		(lib_id "JLC:ME6211C33M5G-N")
+		(lib_id "Parts:ME6211C33M5G-N")
 		(at 330.2 59.69 0)
 		(unit 1)
@@
 			)
 		)
-		(property "Footprint" "JLC:SOT-23-5_L3.0-W1.7-P0.95-LS2.8-BL"
+		(property "Footprint" "Parts:SOT-23-5_L3.0-W1.7-P0.95-LS2.8-BL"
 			(at 330 60 0)
 			(hide yes)
@@
 			)
 		)
-		(property "Footprint" "JLC:LED-SMD_L1.6-W0.8-R-RD"
+		(property "Footprint" "Parts:LED-SMD_L1.6-W0.8-R-RD"
 			(at 162.56 318.77 0)
 			(hide yes)
@@
 			)
 		)
-		(property "Footprint" "JLC:LED-SMD_L1.6-W0.8-R-RD"
+		(property "Footprint" "Parts:LED-SMD_L1.6-W0.8-R-RD"
 			(at 314.96 337.82 0)
 			(hide yes)
@@
 	)
 	(symbol
-		(lib_id "JLC:TS-1187A-B-A-B")
+		(lib_id "Parts:TS-1187A-B-A-B")
 		(at 199.39 149.86 0)
 		(unit 1)
@@
 			)
 		)
-		(property "Footprint" "JLC:SW-SMD_4P-L5.1-W5.1-P3.70-LS6.5-TL_H1.5"
+		(property "Footprint" "Parts:SW-SMD_4P-L5.1-W5.1-P3.70-LS6.5-TL_H1.5"
 			(at 200 150 0)
 			(hide yes)
@@
 			)
 		)
-		(property "Footprint" "JLC:LED-SMD_L1.6-W0.8-R-RD"
+		(property "Footprint" "Parts:LED-SMD_L1.6-W0.8-R-RD"
 			(at 111.76 356.87 0)
 			(hide yes)
@@
 			)
 		)
-		(property "Footprint" "JLC:LED-SMD_L1.6-W0.8-R-RD"
+		(property "Footprint" "Parts:LED-SMD_L1.6-W0.8-R-RD"
 			(at 111.76 337.82 0)
 			(hide yes)
@@
 			)
 		)
-		(property "Footprint" "JLC:LED-SMD_L1.6-W0.8-R-RD"
+		(property "Footprint" "Parts:LED-SMD_L1.6-W0.8-R-RD"
 			(at 213.36 356.87 0)
 			(hide yes)
@@
 			)
 		)
-		(property "Footprint" "JLC:LED-SMD_L1.6-W0.8-R-RD"
+		(property "Footprint" "Parts:LED-SMD_L1.6-W0.8-R-RD"
 			(at 213.36 318.77 0)
 			(hide yes)
@@
 			)
 		)
-		(property "Footprint" "JLC:LED-SMD_L1.6-W0.8-R-RD"
+		(property "Footprint" "Parts:LED-SMD_L1.6-W0.8-R-RD"
 			(at 264.16 318.77 0)
 			(hide yes)
@@
 			)
 		)
-		(property "Footprint" "JLC:LED-SMD_L1.6-W0.8-R-RD"
+		(property "Footprint" "Parts:LED-SMD_L1.6-W0.8-R-RD"
 			(at 264.16 299.72 0)
 			(hide yes)
@@
 	)
 	(symbol
-		(lib_id "JLC:USBLC6-2SC6")
+		(lib_id "Parts:USBLC6-2SC6")
 		(at 261.62 66.04 0)
 		(unit 1)
@@
 			)
 		)
-		(property "Footprint" "JLC:SOT-23-6_L2.9-W1.6-P0.95-LS2.8-BL"
+		(property "Footprint" "Parts:SOT-23-6_L2.9-W1.6-P0.95-LS2.8-BL"
 			(at 262 66 0)
 			(hide yes)
@@
 			)
 		)
-		(property "Footprint" "JLC:LED-SMD_L1.6-W0.8-R-RD"
+		(property "Footprint" "Parts:LED-SMD_L1.6-W0.8-R-RD"
 			(at 60.96 318.77 0)
 			(hide yes)
@@
 			)
 		)
-		(property "Footprint" "JLC:LED-SMD_L1.6-W0.8-R-RD"
+		(property "Footprint" "Parts:LED-SMD_L1.6-W0.8-R-RD"
 			(at 264.16 337.82 0)
 			(hide yes)
@@
 			)
 		)
-		(property "Footprint" "JLC:LED-SMD_L1.6-W0.8-R-RD"
+		(property "Footprint" "Parts:LED-SMD_L1.6-W0.8-R-RD"
 			(at 60.96 299.72 0)
 			(hide yes)
@@
 	)
 	(symbol
-		(lib_id "JLC:LSM6DS3TR-C")
+		(lib_id "Parts:LSM6DS3TR-C")
 		(at 312.42 149.86 0)
 		(unit 1)
@@
 			)
 		)
-		(property "Footprint" "JLC:LGA-14_L3.0-W2.5-P0.50-TL"
+		(property "Footprint" "Parts:LGA-14_L3.0-W2.5-P0.50-TL"
 			(at 312 150 0)
 			(hide yes)
@@
 			)
 		)
-		(property "Footprint" "JLC:LED-SMD_L1.6-W0.8-R-RD"
+		(property "Footprint" "Parts:LED-SMD_L1.6-W0.8-R-RD"
 			(at 314.96 356.87 0)
 			(hide yes)
@@
 			)
 		)
-		(property "Footprint" "JLC:LED-SMD_L1.6-W0.8-R-RD"
+		(property "Footprint" "Parts:LED-SMD_L1.6-W0.8-R-RD"
 			(at 162.56 356.87 0)
 			(hide yes)
@@
 			)
 		)
-		(property "Footprint" "JLC:LED-SMD_L1.6-W0.8-R-RD"
+		(property "Footprint" "Parts:LED-SMD_L1.6-W0.8-R-RD"
 			(at 162.56 337.82 0)
 			(hide yes)
@@
 			)
 		)
-		(property "Footprint" "JLC:LED-SMD_L1.6-W0.8-R-RD"
+		(property "Footprint" "Parts:LED-SMD_L1.6-W0.8-R-RD"
 			(at 111.76 299.72 0)
 			(hide yes)
@@
 	)
 	(symbol
-		(lib_id "JLC:CR2032-BS-6-1")
+		(lib_id "Parts:CR2032-BS-6-1")
 		(at 55.88 73.66 0)
 		(unit 1)
@@
 			)
 		)
-		(property "Footprint" "JLC:BAT-TH_CR2032-BS-6-1"
+		(property "Footprint" "Parts:BAT-TH_CR2032-BS-6-1"
 			(at 55.88 73.66 0)
 			(hide yes)
@@
 			)
 		)
-		(property "Footprint" "JLC:LED-SMD_L1.6-W0.8-R-RD"
+		(property "Footprint" "Parts:LED-SMD_L1.6-W0.8-R-RD"
 			(at 314.96 318.77 0)
 			(hide yes)
@@
 			)
 		)
-		(property "Footprint" "JLC:LED-SMD_L1.6-W0.8-R-RD"
+		(property "Footprint" "Parts:LED-SMD_L1.6-W0.8-R-RD"
 			(at 213.36 337.82 0)
 			(hide yes)
@@
 	)
 	(symbol
-		(lib_id "JLC:TYPE-C-31-M-12")
+		(lib_id "Parts:TYPE-C-31-M-12")
 		(at 185.42 66.04 0)
 		(unit 1)
@@
 			)
 		)
-		(property "Footprint" "JLC:USB-C_SMD-TYPE-C-31-M-12_1"
+		(property "Footprint" "Parts:USB-C_SMD-TYPE-C-31-M-12_1"
 			(at 185 66 0)
 			(hide yes)
@@
 			)
 		)
-		(property "Footprint" "JLC:LED-SMD_L1.6-W0.8-R-RD"
+		(property "Footprint" "Parts:LED-SMD_L1.6-W0.8-R-RD"
 			(at 60.96 356.87 0)
 			(hide yes)
@@
 			)
 		)
-		(property "Footprint" "JLC:LED-SMD_L1.6-W0.8-R-RD"
+		(property "Footprint" "Parts:LED-SMD_L1.6-W0.8-R-RD"
 			(at 60.96 337.82 0)
 			(hide yes)
@@
 			)
 		)
-		(property "Footprint" "JLC:LED-SMD_L1.6-W0.8-R-RD"
+		(property "Footprint" "Parts:LED-SMD_L1.6-W0.8-R-RD"
 			(at 264.16 356.87 0)
 			(hide yes)
@@
 			)
 		)
-		(property "Footprint" "JLC:LED-SMD_L1.6-W0.8-R-RD"
+		(property "Footprint" "Parts:LED-SMD_L1.6-W0.8-R-RD"
 			(at 314.96 299.72 0)
 			(hide yes)
@@
 	)
 	(symbol
-		(lib_id "JLC:AO3401A")
+		(lib_id "Parts:AO3401A")
 		(at 400.05 58.42 0)
 		(unit 1)
@@
 			)
 		)
-		(property "Footprint" "JLC:SOT-23_L2.9-W1.3-P1.90-LS2.4-BR"
+		(property "Footprint" "Parts:SOT-23_L2.9-W1.3-P1.90-LS2.4-BR"
 			(at 400 58 0)
 			(hide yes)
@@
 			)
 		)
-		(property "Footprint" "JLC:LED-SMD_L1.6-W0.8-R-RD"
+		(property "Footprint" "Parts:LED-SMD_L1.6-W0.8-R-RD"
 			(at 213.36 299.72 0)
 			(hide yes)
@@
 			)
 		)
-		(property "Footprint" "JLC:LED-SMD_L1.6-W0.8-R-RD"
+		(property "Footprint" "Parts:LED-SMD_L1.6-W0.8-R-RD"
 			(at 162.56 299.72 0)
 			(hide yes)
@@
 	)
 	(symbol
-		(lib_id "JLC:TS-1187A-B-A-B")
+		(lib_id "Parts:TS-1187A-B-A-B")
 		(at 63.5 149.86 0)
 		(unit 1)
@@
 			)
 		)
-		(property "Footprint" "JLC:SW-SMD_4P-L5.1-W5.1-P3.70-LS6.5-TL_H1.5"
+		(property "Footprint" "Parts:SW-SMD_4P-L5.1-W5.1-P3.70-LS6.5-TL_H1.5"
 			(at 64 150 0)
 			(hide yes)
@@
 			)
 		)
-		(property "Footprint" "JLC:LED-SMD_L1.6-W0.8-R-RD"
+		(property "Footprint" "Parts:LED-SMD_L1.6-W0.8-R-RD"
 			(at 111.76 318.77 0)
 			(hide yes)
@@
 	)
 	(symbol
-		(lib_id "JLC:ESP32-S3-WROOM-1")
+		(lib_id "Parts:ESP32-S3-WROOM-1")
 		(at 129.54 175.26 0)
 		(unit 1)
@@
 			)
 		)
-		(property "Footprint" "JLC:WIRELM-SMD_ESP32-S3-WROOM-1"
+		(property "Footprint" "Parts:WIRELM-SMD_ESP32-S3-WROOM-1"
 			(at 130 175 0)
 			(hide yes)

Commit message: regenerate fab package
Other:
- note added: "IMU"
- note added: "MCU CORE"
- note added: "NEURON LEDs"
- note added: "NFC"
- note added: "POWER"
- note added: "USB-C"
- note removed: "IMU (LSM6DS3TR-C 6-axis, I2C addr 0x6B)"
- note removed: "MCU CORE (ESP32-S3-WROOM-1 + UART programming header)"
- note removed: "NEURON LEDs (24x charlieplex on 6 GPIO) input(6) > hidden(8) > output(10)"
- note removed: "NFC (ST25DV04KC, I2C addr 0x53/0x57, PCB coil on AC0/AC1)"
- note removed: "POWER (CR2032 coin -> SW3 -> VBAT_SW -> Q1 P-FET -> 3V3 rail)"
- note removed: "USB-C (VBUS -> ME6211 3.3V LDO; Q1 P-FET isolates coin when USB present; USBLC6 ESD)"
- moved on the sheet: ANT1, C1, C10, C11, C12, C2, C3, C4, C5, C6, C7, C8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
